Commit message: sim commit

File: src/bdr_ur10_moveit_config/config/gazebo_ur10_description_v3.urdf (robot description, URDF)
Before this commit: robot ur10_description_v3, 12 links, 11 joints
Links:
- added link rgbd_camera_depth_frame, mass 0.001
- added link rgbd_camera_depth_optical_frame, mass 0.001
- added link rgbd_camera_link, mass 0.21970000000; visual box size=0.025 0.1 0.025
- added link rgbd_camera_optical_frame, mass 0.001
- added link rgbd_camera_rgb_frame, mass 0.001
- added link rgbd_camera_rgb_optical_frame, mass 0.001
Joints:
- added joint rgbd_camera_depth_joint: type fixed, parent rgbd_camera_link, child rgbd_camera_depth_frame, origin xyz=0.0 0.049 0.0 rpy=0 0 0
- added joint rgbd_camera_depth_optical_joint: type fixed, parent rgbd_camera_depth_frame, child rgbd_camera_depth_optical_frame, origin xyz=0 0 0 rpy=-1.5707963267948966 0.0 -1.5707963267948966
- added joint rgbd_camera_joint: type fixed, parent camera_link, child rgbd_camera_link, origin xyz=0 0 0 rpy=0 0 -1.57
- added joint rgbd_camera_optical_joint: type fixed, parent rgbd_camera_link, child rgbd_camera_optical_frame, origin xyz=0 0 0 rpy=0 0 -1.57
- added joint rgbd_camera_rgb_joint: type fixed, parent rgbd_camera_link, child rgbd_camera_rgb_frame, origin xyz=0.0 0.022 0.0 rpy=0 0 0
- added joint rgbd_camera_rgb_optical_joint: type fixed, parent rgbd_camera_rgb_frame, child rgbd_camera_rgb_optical_frame, origin xyz=0 0 0 rpy=-1.5707963267948966 0.0 -1.5707963267948966
