Commit message: 23.04 commmit weil Angst

File: src/ur10_description_v3/urdf/ur10_description_v3.urdf (robot description, URDF)
Before this commit: robot ur10_description_v3, 11 links, 10 joints
Joints:
- removed joint motor_1
- removed joint motor_2
- removed joint motor_3
- removed joint motor_4
- removed joint motor_5
- removed joint motor_6
- added joint elbow_joint: type revolute, parent upper_arm_link, child forearm_link, origin xyz=-0.612 0 0 rpy=0 0 0.0242666741712824, axis 0 0 1, limit lower=-3.14 upper=3.14 effort=150 velocity=180
- added joint shoulder_lift_joint: type revolute, parent shoulder_link, child upper_arm_link, origin xyz=0 0.0859989999999999 0.0882571802206784 rpy=1.5707963267949 0.0240929901040578 3.14159265358979, axis 0 0 -1, limit lower=-6.28 upper=6.28 effort=330 velocity=120
- added joint shoulder_pan_joint: type revolute, parent base_link, child shoulder_link, origin xyz=0 0 0.038 rpy=0 0 0, axis 0 0 1, limit lower=-6.28 upper=6.28 effort=330 velocity=120
- added joint wrist_1_joint: type revolute, parent forearm_link, child wrist_1_link, origin xyz=-0.5716 0 0.0220010000000001 rpy=0 0 -0.000173684067224549, axis 0 0 -1, limit lower=-6.28 upper=6.28 effort=56 velocity=180
- added joint wrist_2_joint: type revolute, parent wrist_1_link, child wrist_2_link, origin xyz=0 -0.0617000000000001 0.054 rpy=1.5707963267949 0 0, axis 0 0 -1, limit lower=-6.28 upper=6.28 effort=56 velocity=180
- added joint wrist_3_joint: type revolute, parent wrist_2_link, child wrist_3_link, origin xyz=0 0.0617 0.054 rpy=-1.5707963267949 0.0141025375343068 0, axis 0 0 1, limit lower=-6.28 upper=6.28 effort=56 velocity=180

Commit message: Angst

File: src/ur10_description_v3/urdf/ur10_description_v3.urdf (robot description, URDF)
Before this commit: robot ur10_description_v3, 11 links, 10 joints
Links:
- added link base
Joints:
- added joint base_link-base_fixed_joint: type fixed, parent base_link, child base, origin xyz=0 0 0 rpy=0 0 3.14
- joint shoulder_pan_joint: origin xyz=0 0 0.038 rpy=0 0 0 -> xyz=0 0 0.038 rpy=0 0 -1.57

Commit message: Achsen Negierung negiert

File: src/ur10_description_v3/urdf/ur10_description_v3.urdf (robot description, URDF)
Before this commit: robot ur10_description_v3, 12 links, 11 joints
Links:
- removed link test_finger_link
- added link tool0, mass 0.159494248297753; collision mesh filename=package://ur10_description_v3/meshes/test_finger_link.STL; visual mesh filename=package://ur10_description_v3/meshes/test_finger_link.STL
Joints:
- removed joint tool_test_finger
- added joint tool0: type fixed, parent wrist_3_link, child tool0, origin xyz=0 -0.0486072989450782 0.0984743807368732 rpy=0.785398163397435 0 0, axis 0 0 0
- joint shoulder_lift_joint: axis 0 0 -1 -> 0 0 1
- joint wrist_1_joint: axis 0 0 -1 -> 0 0 1
- joint wrist_2_joint: axis 0 0 -1 -> 0 0 1

Commit message: Koordinatensystem is richtig

File: src/ur10_description_v3/urdf/ur10_description_v3.urdf (robot description, URDF)
Before this commit: robot ur10_description_v3, 12 links, 11 joints
Links:
- removed link tool0
- added link tool0_link, mass 0.159494248297753; collision mesh filename=package://ur10_description_v3/meshes/test_finger_link.STL; visual mesh filename=package://ur10_description_v3/meshes/test_finger_link.STL
Joints:
- joint tool0: child tool0 -> tool0_link

Commit message: Kamera funktioniert

File: src/ur10_description_v3/urdf/ur10_description_v3.urdf (robot description, URDF)
Before this commit: robot ur10_description_v3, 12 links, 11 joints
Links:
- added link camera_config_link, mass 1E-10
Joints:
- added joint camera_config_joint: type fixed, parent camera_link, child camera_config_link, origin xyz=0 0 0 rpy=0 -1.57 -1.57
