Commit message: added quantec, moveit_demo works

File: src/bdr11_description/urdf/ur10_robot.xacro (robot description, xacro)
@@ -9,6 +9,7 @@
     <xacro:include filename="$(find ur10_description_v3)/urdf/kinetic_rgbd.urdf.xacro"/>
     <xacro:include filename="$(find ur10_description_v3)/urdf/kinetic_rgbd.gazebo.xacro"/>
+    <xacro:property name="ur10_ns" value="ur10_" />
     <xacro:macro name="ur10_robot" params="">
-        <link name="table_link">
+        <link name="${ur10_ns}table_link">
             <inertial>
                 <origin xyz="0.503679778923471 0.436750246454337 0.533162239913515" rpy="0 0 0" />
@@ -32,5 +33,5 @@
             </collision>
         </link>
-        <link name="adapter_link">
+        <link name="${ur10_ns}adapter_link">
             <inertial>
                 <origin xyz="0.00148762870939384 -5.55111512312578E-17 0.0184969952138566" rpy="0 0 0" />
@@ -54,11 +55,11 @@
             </collision>
         </link>
-        <joint name="adapter_joint" type="fixed">
+        <joint name="${ur10_ns}adapter_joint" type="fixed">
             <origin xyz="0.17 0.4 0.9" rpy="0 0 0" />
-            <parent link="table_link" />
-            <child link="adapter_link" />
+            <parent link="${ur10_ns}table_link" />
+            <child link="${ur10_ns}adapter_link" />
             <axis xyz="0 0 0" />
         </joint>
-        <link name="base_link">
+        <link name="${ur10_ns}base_link">
             <inertial>
                 <origin xyz="0.0011845 -2.7253E-08 0.017325" rpy="0 0 0" />
@@ -82,11 +83,11 @@
             </collision>
         </link>
-        <joint name="base_joint" type="fixed">
+        <joint name="${ur10_ns}base_joint" type="fixed">
             <origin xyz="0 0 0.037" rpy="0 0 0" />
-            <parent link="adapter_link" />
-            <child link="base_link" />
+            <parent link="${ur10_ns}adapter_link" />
+            <child link="${ur10_ns}base_link" />
             <axis xyz="0 0 0" />
         </joint>
-        <link name="shoulder_link">
+        <link name="${ur10_ns}shoulder_link">
             <inertial>
                 <origin xyz="2.679E-07 0.010024 0.0831" rpy="0 0 0" />
@@ -110,12 +111,12 @@
             </collision>
         </link>
-        <joint name="shoulder_pan_joint" type="revolute">
+        <joint name="${ur10_ns}shoulder_pan_joint" type="revolute">
             <origin xyz="0 0 0.038" rpy="0 0 -1.57" />
-            <parent link="base_link" />
-            <child link="shoulder_link" />
+            <parent link="${ur10_ns}base_link" />
+            <child link="${ur10_ns}shoulder_link" />
             <axis xyz="0 0 1" />
             <limit lower="-6.28" upper="6.28" effort="330" velocity="120" />
         </joint>
-        <link name="upper_arm_link">
+        <link name="${ur10_ns}upper_arm_link">
             <inertial>
                 <origin xyz="-0.25443 -2.027E-07 0.082537" rpy="0 0 0" />
@@ -139,12 +140,12 @@
             </collision>
         </link>
-        <joint name="shoulder_lift_joint" type="revolute">
+        <joint name="${ur10_ns}shoulder_lift_joint" type="revolute">
             <origin xyz="0 0.0859989999999999 0.0882571802206784" rpy="1.5707963267949 0.0240929901040578 3.14159265358979" />
-            <parent link="shoulder_link" />
-            <child link="upper_arm_link" />
+            <parent link="${ur10_ns}shoulder_link" />
+            <child link="${ur10_ns}upper_arm_link" />
             <axis xyz="0 0 1" />
             <limit lower="-6.28" upper="6.28" effort="330" velocity="120" />
         </joint>
-        <link name="forearm_link">
+        <link name="${ur10_ns}forearm_link">
             <inertial>
                 <origin xyz="-0.24807 1.9251E-09 -0.034936" rpy="0 0 0" />
@@ -168,12 +169,12 @@
             </collision>
         </link>
-        <joint name="elbow_joint" type="revolute">
+        <joint name="${ur10_ns}elbow_joint" type="revolute">
             <origin xyz="-0.612 0 0" rpy="0 0 0.0242666741712824" />
-            <parent link="upper_arm_link" />
-            <child link="forearm_link" />
+            <parent link="${ur10_ns}upper_arm_link" />
+            <child link="${ur10_ns}forearm_link" />
             <axis xyz="0 0 1" />
             <limit lower="-3.14" upper="3.14" effort="150" velocity="180" />
         </joint>
-        <link name="wrist_1_link">
+        <link name="${ur10_ns}wrist_1_link">
             <inertial>
                 <origin xyz="8.3814E-09 -0.010045 0.046994" rpy="0 0 0" />
@@ -197,12 +198,12 @@
             </collision>
         </link>
-        <joint name="wrist_1_joint" type="revolute">
+        <joint name="${ur10_ns}wrist_1_joint" type="revolute">
             <origin xyz="-0.5716 0 0.0220010000000001" rpy="0 0 -0.000173684067224549" />
-            <parent link="forearm_link" />
-            <child link="wrist_1_link" />
+            <parent link="${ur10_ns}forearm_link" />
+            <child link="${ur10_ns}wrist_1_link" />
             <axis xyz="0 0 1" />
             <limit lower="-6.28" upper="6.28" effort="56" velocity="180" />
         </joint>
-        <link name="wrist_2_link">
+        <link name="${ur10_ns}wrist_2_link">
             <inertial>
                 <origin xyz="-8.3814E-09 0.010045 0.046994" rpy="0 0 0" />
@@ -226,12 +227,12 @@
             </collision>
         </link>
-        <joint name="wrist_2_joint" type="revolute">
+        <joint name="${ur10_ns}wrist_2_joint" type="revolute">
             <origin xyz="0 -0.0617000000000001 0.054" rpy="1.5707963267949 0 0" />
-            <parent link="wrist_1_link" />
-            <child link="wrist_2_link" />
+            <parent link="${ur10_ns}wrist_1_link" />
+            <child link="${ur10_ns}wrist_2_link" />
             <axis xyz="0 0 1" />
             <limit lower="-6.28" upper="6.28" effort="56" velocity="180" />
         </joint>
-        <link name="wrist_3_link">
+        <link name="${ur10_ns}wrist_3_link">
             <inertial>
                 <origin xyz="2.2204E-16 -1.1102E-16 0.015005" rpy="0 0 0" />
@@ -255,12 +256,12 @@
             </collision>
         </link>
-        <joint name="wrist_3_joint" type="revolute">
+        <joint name="${ur10_ns}wrist_3_joint" type="revolute">
             <origin xyz="0 0.0617 0.054" rpy="-1.5707963267949 0.0141025375343068 0" />
-            <parent link="wrist_2_link" />
-            <child link="wrist_3_link" />
+            <parent link="${ur10_ns}wrist_2_link" />
+            <child link="${ur10_ns}wrist_3_link" />
             <axis xyz="0 0 1" />
             <limit lower="-6.28" upper="6.28" effort="56" velocity="180" />
         </joint>
-        <link name="tool0_link">
+        <link name="${ur10_ns}tool0_link">
             <inertial>
                 <origin xyz="-9.51811385263568E-09 -0.00040829549117638 -0.063076624107084" rpy="0 0 0" />
@@ -284,11 +285,11 @@
             </collision>
         </link>
-        <joint name="tool0" type="fixed">
+        <joint name="${ur10_ns}tool0" type="fixed">
             <origin xyz="0 -0.0486072989450782 0.0984743807368732" rpy="0.785398163397435 0 0" />
-            <parent link="wrist_3_link" />
-            <child link="tool0_link" />
+            <parent link="${ur10_ns}wrist_3_link" />
+            <child link="${ur10_ns}tool0_link" />
             <axis xyz="0 0 0" />
         </joint>
-        <link name="camera_link">
+        <link name="${ur10_ns}camera_link">
             <inertial>
                 <origin xyz="-1.61524861117535E-05 -0.00212700504491092 -0.0193765848255853" rpy="0 0 0" />
@@ -312,66 +313,66 @@
             </collision>
         </link>
-        <joint name="tool_camera" type="fixed">
+        <joint name="${ur10_ns}tool_camera" type="fixed">
             <origin xyz="0 0.0158483827537649 0.0919267022436815" rpy="0.856180071631976 0 0" />
-            <parent link="wrist_3_link" />
-            <child link="camera_link" />
+            <parent link="${ur10_ns}wrist_3_link" />
+            <child link="${ur10_ns}camera_link" />
             <axis xyz="0 0 0" />
         </joint>
-        <transmission name="trans_shoulder_pan_joint">
-            <type>transmission_interface/SimpleTransmission</type>
-            <joint name="shoulder_pan_joint">
-                <hardwareInterface>hardware_interface/EffortJointInterface</hardwareInterface>
-            </joint>
-            <actuator name="shoulder_pan_joint_motor">
-                <hardwareInterface>hardware_interface/EffortJointInterface</hardwareInterface>
-                <mechanicalReduction>1</mechanicalReduction>
-            </actuator>
-        </transmission>
-        <transmission name="trans_shoulder_lift_joint">
-            <type>transmission_interface/SimpleTransmission</type>
-            <joint name="shoulder_lift_joint">
-                <hardwareInterface>hardware_interface/EffortJointInterface</hardwareInterface>
-            </joint>
-            <actuator name="shoulder_lift_joint_motor">
-                <hardwareInterface>hardware_interface/EffortJointInterface</hardwareInterface>
-                <mechanicalReduction>1</mechanicalReduction>
-            </actuator>
-        </transmission>
-        <transmission name="trans_elbow_joint">
-            <type>transmission_interface/SimpleTransmission</type>
-            <joint name="elbow_joint">
-                <hardwareInterface>hardware_interface/EffortJointInterface</hardwareInterface>
-            </joint>
-            <actuator name="elbow_joint_motor">
-                <hardwareInterface>hardware_interface/EffortJointInterface</hardwareInterface>
-                <mechanicalReduction>1</mechanicalReduction>
-            </actuator>
-        </transmission>
-        <transmission name="trans_wrist_1_joint">
-            <type>transmission_interface/SimpleTransmission</type>
-            <joint name="wrist_1_joint">
-                <hardwareInterface>hardware_interface/EffortJointInterface</hardwareInterface>
-            </joint>
-            <actuator name="wrist_1_joint_motor">
-                <hardwareInterface>hardware_interface/EffortJointInterface</hardwareInterface>
-                <mechanicalReduction>1</mechanicalReduction>
-            </actuator>
-        </transmission>
-        <transmission name="trans_wrist_2_joint">
-            <type>transmission_interface/SimpleTransmission</type>
-            <joint name="wrist_2_joint">
-                <hardwareInterface>hardware_interface/EffortJointInterface</hardwareInterface>
-            </joint>
-            <actuator name="wrist_2_joint_motor">
-                <hardwareInterface>hardware_interface/EffortJointInterface</hardwareInterface>
-                <mechanicalReduction>1</mechanicalReduction>
-            </actuator>
-        </transmission>
-        <transmission name="trans_wrist_3_joint">
-            <type>transmission_interface/SimpleTransmission</type>
-            <joint name="wrist_3_joint">
-                <hardwareInterface>hardware_interface/EffortJointInterface</hardwareInterface>
-            </joint>
-            <actuator name="wrist_3_joint_motor">
+        <transmission name="${ur10_ns}trans_shoulder_pan_joint">
+            <type>transmission_interface/SimpleTransmission</type>
+            <joint name="${ur10_ns}shoulder_pan_joint">
+                <hardwareInterface>hardware_interface/EffortJointInterface</hardwareInterface>
+            </joint>
+            <actuator name="${ur10_ns}shoulder_pan_joint_motor">
+                <hardwareInterface>hardware_interface/EffortJointInterface</hardwareInterface>
+                <mechanicalReduction>1</mechanicalReduction>
+            </actuator>
+        </transmission>
+        <transmission name="${ur10_ns}trans_shoulder_lift_joint">
+            <type>transmission_interface/SimpleTransmission</type>
+            <joint name="${ur10_ns}shoulder_lift_joint">
+                <hardwareInterface>hardware_interface/EffortJointInterface</hardwareInterface>
+            </joint>
+            <actuator name="${ur10_ns}shoulder_lift_joint_motor">
+                <hardwareInterface>hardware_interface/EffortJointInterface</hardwareInterface>
+                <mechanicalReduction>1</mechanicalReduction>
+            </actuator>
+        </transmission>
+        <transmission name="${ur10_ns}trans_elbow_joint">
+            <type>transmission_interface/SimpleTransmission</type>
+            <joint name="${ur10_ns}elbow_joint">
+                <hardwareInterface>hardware_interface/EffortJointInterface</hardwareInterface>
+            </joint>
+            <actuator name="${ur10_ns}elbow_joint_motor">
+                <hardwareInterface>hardware_interface/EffortJointInterface</hardwareInterface>
+                <mechanicalReduction>1</mechanicalReduction>
+            </actuator>
+        </transmission>
+        <transmission name="${ur10_ns}trans_wrist_1_joint">
+            <type>transmission_interface/SimpleTransmission</type>
+            <joint name="${ur10_ns}wrist_1_joint">
+                <hardwareInterface>hardware_interface/EffortJointInterface</hardwareInterface>
+            </joint>
+            <actuator name="${ur10_ns}wrist_1_joint_motor">
+                <hardwareInterface>hardware_interface/EffortJointInterface</hardwareInterface>
+                <mechanicalReduction>1</mechanicalReduction>
+            </actuator>
+        </transmission>
+        <transmission name="${ur10_ns}trans_wrist_2_joint">
+            <type>transmission_interface/SimpleTransmission</type>
+            <joint name="${ur10_ns}wrist_2_joint">
+                <hardwareInterface>hardware_interface/EffortJointInterface</hardwareInterface>
+            </joint>
+            <actuator name="${ur10_ns}wrist_2_joint_motor">
+                <hardwareInterface>hardware_interface/EffortJointInterface</hardwareInterface>
+                <mechanicalReduction>1</mechanicalReduction>
+            </actuator>
+        </transmission>
+        <transmission name="${ur10_ns}trans_wrist_3_joint">
+            <type>transmission_interface/SimpleTransmission</type>
+            <joint name="${ur10_ns}wrist_3_joint">
+                <hardwareInterface>hardware_interface/EffortJointInterface</hardwareInterface>
+            </joint>
+            <actuator name="${ur10_ns}wrist_3_joint_motor">
                 <hardwareInterface>hardware_interface/EffortJointInterface</hardwareInterface>
                 <mechanicalReduction>1</mechanicalReduction>
@@ -379,7 +380,7 @@
         </transmission>
         <!-- force/torque sensor -->
-        <xacro:ft_sensor_gazebo joint="wrist_3_joint"/>
+        <xacro:ft_sensor_gazebo joint="${ur10_ns}wrist_3_joint"/>
         <!-- camera -->
-        <xacro:kinetic_rgb name="rgbd_camera" parent="camera">
+        <xacro:kinetic_rgb name="rgbd_camera" parent="${ur10_ns}camera">
             <origin xyz="0 0 0.005" rpy="0 0 3.14"/>
             <origin xyz="0 0 0" rpy="0 0 0"/>
@@ -387,10 +388,10 @@
         <gazebo>
         <plugin name="gazebo_ros_control" filename="libgazebo_ros_control.so">
-            <!-- <robotNamespace></robotNamespace> -->
+            <robotNamespace>$/{ur10_ns}</robotNamespace>
         </plugin>
         </gazebo>
         <!-- ROS-Industrial 'base' frame: base_link to UR 'Base' Coordinates transform -->
-        <link name="base"/>
-        <joint name="base_link-base_fixed_joint" type="fixed">
+        <link name="${ur10_ns}base"/>
+        <joint name="${ur10_ns}base_link-base_fixed_joint" type="fixed">
         <!-- Note the rotation over Z of pi radians: as base_link is REP-103
             aligned (ie: has X+ forward, Y+ left and Z+ up), this is needed
@@ -399,9 +400,9 @@
         -->
         <origin xyz="0 0 0" rpy="0 0 3.14"/>
-        <parent link="base_link"/>
-        <child link="base"/>
+        <parent link="${ur10_ns}base_link"/>
+        <child link="${ur10_ns}base"/>
         </joint>
     </xacro:macro>
     <!-- call -->
-    <xacro:ur10_robot/>
+    <!-- <xacro:ur10_robot/> -->
 </robot>

File: src/ur10_description_v3/urdf/kinetic_rgbd.urdf.xacro (robot description, xacro)
@@ -52,5 +52,5 @@
         <!-- Depth sensor frames -->
         <joint name="${name}_depth_joint" type="fixed">
-            <origin xyz="0.049 0.0 0.0" rpy="0 0 0"/>   <!--origin xyz="0.0 0.049 0.0" rpy="0 0 0"-->
+            <origin xyz="-0.025 0.0 0.0" rpy="1.57 -1.57 0"/>   <!--origin xyz="0.0 0.049 0.0" rpy="0 0 0"-->
             <parent link="${name}_link"/>
             <child link="${name}_depth_frame"/>
@@ -60,5 +60,5 @@
         </link>
         <joint name="${name}_depth_optical_joint" type="fixed">
-            <origin xyz="0 0 0" rpy="${0 * deg_to_rad} 0.0 ${0 * deg_to_rad}"/>  <!-- -90 deg_to_rad - x&z -->
+            <origin xyz="0 0 0" rpy="${-90 * deg_to_rad} 0.0 ${-90 * deg_to_rad}"/>  <!-- -90 deg_to_rad - x&z -->
             <parent link="${name}_depth_frame"/>
             <child link="${name}_depth_optical_frame"/>
@@ -69,5 +69,5 @@
         <!-- RGB sensor frames -->
         <joint name="${name}_rgb_joint" type="fixed">
-            <origin xyz="0.0 0.022 0.0" rpy="0 0 0"/>
+            <origin xyz="0 0 0" rpy="1.57 -1.57 0"/>
             <parent link="${name}_link"/>
             <child link="${name}_rgb_frame"/>
@@ -77,5 +77,5 @@
         </link>
         <joint name="${name}_rgb_optical_joint" type="fixed">
-            <origin xyz="0 0 0" rpy="${0 * deg_to_rad} 0.0 ${0 * deg_to_rad}"/> <!-- -90 deg_to_rad - x&z -->
+            <origin xyz="0 0 0" rpy="${-90 * deg_to_rad} 0.0 ${-90 * deg_to_rad}"/> <!-- -90 deg_to_rad - x&z -->
             <parent link="${name}_rgb_frame"/>
             <child link="${name}_rgb_optical_frame"/>
