Commit message: working gazebo simulation

File: src/bdr11_description/urdf/bdr11.urdf.xacro (robot description, xacro)
@@ -2,23 +2,24 @@
 <robot xmlns:xacro="http://ros.org/wiki/xacro" name="dual_robots">
   <!-- Define the world link -->
-  <link name="world_link">
+  <link name="dual_robot_link">
     <inertial>
       <mass value="1.0" />
-      <origin xyz="0 0 0" rpy="0 0 0" />
+      <origin xyz="0 0 0.0" rpy="0 0 0" /> <!-- Raise the link by changing the z-value -->
       <inertia ixx="0" ixy="0" ixz="0" iyy="0" iyz="0" izz="0" />
     </inertial>
     <visual>
       <geometry>
-        <box size="0.1 0.1 0.1" />
+        <box size="0.01 0.01 0.01" />
       </geometry>
+      <collision>
+          <origin rpy="0 0 0" xyz="0 0 0" />
+          <geometry>
+              <box size="0.01 0.01 0.01" />
+          </geometry>
+      </collision>
       <material name="gray">
         <color rgba="0.5 0.5 0.5 1.0" />
       </material>
     </visual>
-    <collision>
-      <geometry>
-        <box size="0.1 0.1 0.1" />
-      </geometry>
-    </collision>
   </link>
   <!-- First robot -->
@@ -26,7 +27,7 @@
   <xacro:ur10_robot />
   <joint name="ur10_robot_joint" type="fixed">
-    <parent link="world_link" />
-    <child link="${ur10_ns}table_link" />
-    <origin xyz="0 0 0" rpy="0 0 0" />
+    <parent link="dual_robot_link" />
+    <child link="${ur10_ns}table_link" /> <!-- ${ur10_ns} -->
+    <origin xyz="0 0 -0.005" rpy="0 0 0" />
   </joint>
   <!-- Second robot -->
@@ -34,7 +35,7 @@
   <xacro:moveit_quantec />
   <joint name="quantec_robot_joint" type="fixed">
-    <parent link="world_link" />
-    <child link="${quantec_ns}base_link_quantec" />
-    <origin xyz="-1 0.4 0" rpy="-1.57 0 0" /> <!-- Adjust xyz for the desired position -->
+    <parent link="dual_robot_link" />
+    <child link="${quantec_ns}base_link_quantec" />  <!-- ${quantec_ns} -->
+    <origin xyz="-1 0.4 -0.005" rpy="-1.57 0 0" /> <!-- Adjust xyz for the desired position -->
   </joint>
 </robot>

File: src/bdr11_description/urdf/quantec_eff.urdf.xacro (robot description, xacro)
@@ -8,5 +8,5 @@
      For more information, please see http://wiki.ros.org/sw_urdf_exporter -->
 <robot name="moveit_quantec" xmlns:xacro="http://ros.org/wiki/xacro">
-    <xacro:property name="quantec_ns" value="quantec_" />
+    <xacro:property name="quantec_ns" value="" />
     <xacro:macro name="moveit_quantec" params="">
         <link name="${quantec_ns}base_link_quantec">
@@ -200,69 +200,4 @@
             <axis xyz="1 0 0" />
         </joint>
-        <transmission name="${quantec_ns}trans_joint_1">
-            <type>transmission_interface/SimpleTransmission</type>
-            <joint name="${quantec_ns}joint_1">
-                <hardwareInterface>hardware_interface/EffortJointInterface</hardwareInterface>
-            </joint>
-            <actuator name="${quantec_ns}joint_1_motor">
-                <hardwareInterface>hardware_interface/EffortJointInterface</hardwareInterface>
-                <mechanicalReduction>1</mechanicalReduction>
-            </actuator>
-        </transmission>
-        <transmission name="${quantec_ns}trans_joint_2">
-            <type>transmission_interface/SimpleTransmission</type>
-            <joint name="${quantec_ns}joint_2">
-                <hardwareInterface>hardware_interface/EffortJointInterface</hardwareInterface>
-            </joint>
-            <actuator name="${quantec_ns}joint_2_motor">
-                <hardwareInterface>hardware_interface/EffortJointInterface</hardwareInterface>
-                <mechanicalReduction>1</mechanicalReduction>
-            </actuator>
-        </transmission>
-        <transmission name="${quantec_ns}trans_joint_3">
-            <type>transmission_interface/SimpleTransmission</type>
-            <joint name="${quantec_ns}joint_3">
-                <hardwareInterface>hardware_interface/EffortJointInterface</hardwareInterface>
-            </joint>
-            <actuator name="${quantec_ns}joint_3_motor">
-                <hardwareInterface>hardware_interface/EffortJointInterface</hardwareInterface>
-                <mechanicalReduction>1</mechanicalReduction>
-            </actuator>
-        </transmission>
-        <transmission name="${quantec_ns}trans_joint_4">
-            <type>transmission_interface/SimpleTransmission</type>
-            <joint name="joint_4">
-                <hardwareInterface>hardware_interface/EffortJointInterface</hardwareInterface>
-            </joint>
-            <actuator name="${quantec_ns}joint_4_motor">
-                <hardwareInterface>hardware_interface/EffortJointInterface</hardwareInterface>
-                <mechanicalReduction>1</mechanicalReduction>
-            </actuator>
-        </transmission>
-        <transmission name="${quantec_ns}trans_joint_5">
-            <type>transmission_interface/SimpleTransmission</type>
-            <joint name="${quantec_ns}joint_5">
-                <hardwareInterface>hardware_interface/EffortJointInterface</hardwareInterface>
-            </joint>
-            <actuator name="${quantec_ns}joint_5_motor">
-                <hardwareInterface>hardware_interface/EffortJointInterface</hardwareInterface>
-                <mechanicalReduction>1</mechanicalReduction>
-            </actuator>
-        </transmission>
-        <transmission name="${quantec_ns}trans_joint_6">
-            <type>transmission_interface/SimpleTransmission</type>
-            <joint name="${quantec_ns}joint_6">
-                <hardwareInterface>hardware_interface/EffortJointInterface</hardwareInterface>
-            </joint>
-            <actuator name="${quantec_ns}joint_6_motor">
-                <hardwareInterface>hardware_interface/EffortJointInterface</hardwareInterface>
-                <mechanicalReduction>1</mechanicalReduction>
-            </actuator>
-        </transmission>
-        <gazebo>
-            <plugin name="gazebo_ros_control" filename="libgazebo_ros_control.so">
-                <robotNamespace>$/{quantec_ns}</robotNamespace>
-            </plugin>
-        </gazebo>
     </xacro:macro>
     <!-- call -->

File: src/bdr11_description/urdf/ur10_robot.xacro (robot description, xacro)
@@ -9,5 +9,5 @@
     <xacro:include filename="$(find ur10_description_v3)/urdf/kinetic_rgbd.urdf.xacro"/>
     <xacro:include filename="$(find ur10_description_v3)/urdf/kinetic_rgbd.gazebo.xacro"/>
-    <xacro:property name="ur10_ns" value="ur10_" />
+    <xacro:property name="ur10_ns" value="" />
     <xacro:macro name="ur10_robot" params="">
         <link name="${ur10_ns}table_link">
@@ -319,64 +319,4 @@
             <axis xyz="0 0 0" />
         </joint>
-        <transmission name="${ur10_ns}trans_shoulder_pan_joint">
-            <type>transmission_interface/SimpleTransmission</type>
-            <joint name="${ur10_ns}shoulder_pan_joint">
-                <hardwareInterface>hardware_interface/EffortJointInterface</hardwareInterface>
-            </joint>
-            <actuator name="${ur10_ns}shoulder_pan_joint_motor">
-                <hardwareInterface>hardware_interface/EffortJointInterface</hardwareInterface>
-                <mechanicalReduction>1</mechanicalReduction>
-            </actuator>
-        </transmission>
-        <transmission name="${ur10_ns}trans_shoulder_lift_joint">
-            <type>transmission_interface/SimpleTransmission</type>
-            <joint name="${ur10_ns}shoulder_lift_joint">
-                <hardwareInterface>hardware_interface/EffortJointInterface</hardwareInterface>
-            </joint>
-            <actuator name="${ur10_ns}shoulder_lift_joint_motor">
-                <hardwareInterface>hardware_interface/EffortJointInterface</hardwareInterface>
-                <mechanicalReduction>1</mechanicalReduction>
-            </actuator>
-        </transmission>
-        <transmission name="${ur10_ns}trans_elbow_joint">
-            <type>transmission_interface/SimpleTransmission</type>
-            <joint name="${ur10_ns}elbow_joint">
-                <hardwareInterface>hardware_interface/EffortJointInterface</hardwareInterface>
-            </joint>
-            <actuator name="${ur10_ns}elbow_joint_motor">
-                <hardwareInterface>hardware_interface/EffortJointInterface</hardwareInterface>
-                <mechanicalReduction>1</mechanicalReduction>
-            </actuator>
-        </transmission>
-        <transmission name="${ur10_ns}trans_wrist_1_joint">
-            <type>transmission_interface/SimpleTransmission</type>
-            <joint name="${ur10_ns}wrist_1_joint">
-                <hardwareInterface>hardware_interface/EffortJointInterface</hardwareInterface>
-            </joint>
-            <actuator name="${ur10_ns}wrist_1_joint_motor">
-                <hardwareInterface>hardware_interface/EffortJointInterface</hardwareInterface>
-                <mechanicalReduction>1</mechanicalReduction>
-            </actuator>
-        </transmission>
-        <transmission name="${ur10_ns}trans_wrist_2_joint">
-            <type>transmission_interface/SimpleTransmission</type>
-            <joint name="${ur10_ns}wrist_2_joint">
-                <hardwareInterface>hardware_interface/EffortJointInterface</hardwareInterface>
-            </joint>
-            <actuator name="${ur10_ns}wrist_2_joint_motor">
-                <hardwareInterface>hardware_interface/EffortJointInterface</hardwareInterface>
-                <mechanicalReduction>1</mechanicalReduction>
-            </actuator>
-        </transmission>
-        <transmission name="${ur10_ns}trans_wrist_3_joint">
-            <type>transmission_interface/SimpleTransmission</type>
-            <joint name="${ur10_ns}wrist_3_joint">
-                <hardwareInterface>hardware_interface/EffortJointInterface</hardwareInterface>
-            </joint>
-            <actuator name="${ur10_ns}wrist_3_joint_motor">
-                <hardwareInterface>hardware_interface/EffortJointInterface</hardwareInterface>
-                <mechanicalReduction>1</mechanicalReduction>
-            </actuator>
-        </transmission>
         <!-- force/torque sensor -->
         <xacro:ft_sensor_gazebo joint="${ur10_ns}wrist_3_joint"/>
@@ -386,9 +326,4 @@
             <origin xyz="0 0 0" rpy="0 0 0"/>
         </xacro:kinetic_rgb>
-        <gazebo>
-        <plugin name="gazebo_ros_control" filename="libgazebo_ros_control.so">
-            <robotNamespace>$/{ur10_ns}</robotNamespace>    <!--value="ur10_"-->
-        </plugin>
-        </gazebo>
         <!-- ROS-Industrial 'base' frame: base_link to UR 'Base' Coordinates transform -->
         <link name="${ur10_ns}base"/>

File: src/bdr11_moveit_config/config/gazebo_dual_robots.urdf (robot description, URDF)
Before this commit: robot dual_robots, 26 links, 25 joints
Links:
- removed link quantec_base_link_quantec
- removed link quantec_link_1
- removed link quantec_link_2
- removed link quantec_link_3
- removed link quantec_link_4
- removed link quantec_link_5
- removed link quantec_link_6
- removed link ur10_adapter_link
- removed link ur10_base
- removed link ur10_base_link
- removed link ur10_camera_link
- removed link ur10_forearm_link
- removed link ur10_shoulder_link
- removed link ur10_table_link
- removed link ur10_tool0_link
- removed link ur10_upper_arm_link
- removed link ur10_wrist_1_link
- removed link ur10_wrist_2_link
- removed link ur10_wrist_3_link
- removed link world_link
- added link adapter_link, mass 1.3940393775037; collision mesh filename=package://ur10_description_v3/meshes/adapter_link.STL; visual mesh filename=package://ur10_description_v3/meshes/adapter_link.STL
- added link base
- added link base_link, mass 0.86268; collision mesh filename=package://ur10_description_v3/meshes/base_link.STL; visual mesh filename=package://ur10_description_v3/meshes/base_link.STL
- added link base_link_quantec, mass 97.9298238151877; collision mesh filename=package://moveit_quantec/meshes/base_link.STL; visual mesh filename=package://moveit_quantec/meshes/base_link.STL
- added link camera_link, mass 0.0840231018507497; collision mesh filename=package://ur10_description_v3/meshes/camera_link.STL
- added link dual_robot_link, mass 1.0; visual box size=0.01 0.01 0.01
- added link forearm_link, mass 3.87; collision mesh filename=package://ur10_description_v3/meshes/forearm_link.STL; visual mesh filename=package://ur10_description_v3/meshes/forearm_link.STL
- added link link_1, mass 94.945; collision mesh filename=package://moveit_quantec/meshes/link_1.STL; visual mesh filename=package://moveit_quantec/meshes/link_1.STL
- added link link_2, mass 82.176; collision mesh filename=package://moveit_quantec/meshes/link_2.STL; visual mesh filename=package://moveit_quantec/meshes/link_2.STL
- added link link_3, mass 47.124; collision mesh filename=package://moveit_quantec/meshes/link_3.STL; visual mesh filename=package://moveit_quantec/meshes/link_3.STL
- added link link_4, mass 4.6744; collision mesh filename=package://moveit_quantec/meshes/link_4.STL; visual mesh filename=package://moveit_quantec/meshes/link_4.STL
- added link link_5, mass 8.3467; collision mesh filename=package://moveit_quantec/meshes/link_5.STL; visual mesh filename=package://moveit_quantec/meshes/link_5.STL
- added link link_6, mass 0.97276; collision mesh filename=package://moveit_quantec/meshes/link_6.STL; visual mesh filename=package://moveit_quantec/meshes/link_6.STL
- added link shoulder_link, mass 7.778; collision mesh filename=package://ur10_description_v3/meshes/shoulder_link.STL; visual mesh filename=package://ur10_description_v3/meshes/shoulder_link.STL
- added link table_link, mass 164.427518164029; collision mesh filename=package://ur10_description_v3/meshes/table_link.STL; visual mesh filename=package://ur10_description_v3/meshes/table_link.STL
- added link tool0_link, mass 0.159494248297753; collision mesh filename=package://ur10_description_v3/meshes/test_finger_link.STL; visual mesh filename=package://ur10_description_v3/meshes/test_finger_link.STL
- added link upper_arm_link, mass 12.93; collision mesh filename=package://ur10_description_v3/meshes/upper_arm_link.STL; visual mesh filename=package://ur10_description_v3/meshes/upper_arm_link.STL
- added link wrist_1_link, mass 1.96; collision mesh filename=package://ur10_description_v3/meshes/wrist_1_link.STL; visual mesh filename=package://ur10_description_v3/meshes/wrist_1_link.STL
- added link wrist_2_link, mass 1.96; collision mesh filename=package://ur10_description_v3/meshes/wrist_2_link.STL; visual mesh filename=package://ur10_description_v3/meshes/wrist_2_link.STL
- added link wrist_3_link, mass 0.202; collision mesh filename=package://ur10_description_v3/meshes/wrist_3_link.STL; visual mesh filename=package://ur10_description_v3/meshes/wrist_3_link.STL
Joints:
- removed joint quantec_joint_1
- removed joint quantec_joint_2
- removed joint quantec_joint_3
- removed joint quantec_joint_4
- removed joint quantec_joint_5
- removed joint quantec_joint_6
- removed joint ur10_adapter_joint
- removed joint ur10_base_joint
- removed joint ur10_base_link-base_fixed_joint
- removed joint ur10_elbow_joint
- removed joint ur10_shoulder_lift_joint
- removed joint ur10_shoulder_pan_joint
- removed joint ur10_tool0
- removed joint ur10_tool_camera
- removed joint ur10_wrist_1_joint
- removed joint ur10_wrist_2_joint
- removed joint ur10_wrist_3_joint
- added joint adapter_joint: type fixed, parent table_link, child adapter_link, origin xyz=0.17 0.4 0.9 rpy=0 0 0, axis 0 0 0
- added joint base_joint: type fixed, parent adapter_link, child base_link, origin xyz=0 0 0.037 rpy=0 0 0, axis 0 0 0
- added joint base_link-base_fixed_joint: type fixed, parent base_link, child base, origin xyz=0 0 0 rpy=0 0 3.14
- added joint elbow_joint: type revolute, parent upper_arm_link, child forearm_link, origin xyz=-0.612 0 0 rpy=0 0 0.0242666741712824, axis 0 0 1, limit lower=-3.14 upper=3.14 effort=150 velocity=180
- added joint joint_1: type continuous, parent base_link_quantec, child link_1, origin xyz=0 -0.235 0 rpy=1.5708 0.014047 0, axis 0 0 1
- added joint joint_2: type continuous, parent link_1, child link_2, origin xyz=0.33 0 0.41772 rpy=0 -0.0391 0, axis 0 1 0
- added joint joint_3: type continuous, parent link_2, child link_3, origin xyz=0 0 1.15 rpy=0 -0.52738 0, axis 0 1 0
- added joint joint_4: type continuous, parent link_3, child link_4, origin xyz=0.78147 -0.0086752 0.115 rpy=0.037095 0 0, axis 1 0 0
- added joint joint_5: type continuous, parent link_4, child link_5, origin xyz=0.44853 0 0 rpy=0 0.9269 0, axis 0 1 0
- added joint joint_6: type continuous, parent link_5, child link_6, origin xyz=0.20228 1.3733E-05 0 rpy=-2.218 0 0, axis 1 0 0
- added joint shoulder_lift_joint: type revolute, parent shoulder_link, child upper_arm_link, origin xyz=0 0.0859989999999999 0.0882571802206784 rpy=1.5707963267949 0.0240929901040578 3.14159265358979, axis 0 0 1, limit lower=-6.28 upper=6.28 effort=330 velocity=120
- added joint shoulder_pan_joint: type revolute, parent base_link, child shoulder_link, origin xyz=0 0 0.038 rpy=0 0 -1.57, axis 0 0 1, limit lower=-6.28 upper=6.28 effort=330 velocity=120
- added joint tool0: type fixed, parent wrist_3_link, child tool0_link, origin xyz=0 -0.0486072989450782 0.0984743807368732 rpy=0.785398163397435 0 0, axis 0 0 0
- added joint tool_camera: type fixed, parent wrist_3_link, child camera_link, origin xyz=0 0.0158483827537649 0.0919267022436815 rpy=0.856180071631976 0 0, axis 0 0 0
- added joint wrist_1_joint: type revolute, parent forearm_link, child wrist_1_link, origin xyz=-0.5716 0 0.0220010000000001 rpy=0 0 -0.000173684067224549, axis 0 0 1, limit lower=-6.28 upper=6.28 effort=56 velocity=180
- added joint wrist_2_joint: type revolute, parent wrist_1_link, child wrist_2_link, origin xyz=0 -0.0617000000000001 0.054 rpy=1.5707963267949 0 0, axis 0 0 1, limit lower=-6.28 upper=6.28 effort=56 velocity=180
- added joint wrist_3_joint: type revolute, parent wrist_2_link, child wrist_3_link, origin xyz=0 0.0617 0.054 rpy=-1.5707963267949 0.0141025375343068 0, axis 0 0 1, limit lower=-6.28 upper=6.28 effort=56 velocity=180
- joint quantec_robot_joint: child quantec_base_link_quantec -> base_link_quantec; origin xyz=-1 0.4 0 rpy=-1.57 0 0 -> xyz=-1 0.4 -0.005 rpy=-1.57 0 0; parent world_link -> dual_robot_link
- joint rgbd_camera_joint: parent ur10_camera_link -> camera_link
- joint ur10_robot_joint: child ur10_table_link -> table_link; origin xyz=0 0 0 rpy=0 0 0 -> xyz=0 0 -0.005 rpy=0 0 0; parent world_link -> dual_robot_link

Commit message: working PoseArray navigation

File: src/bdr11_description/urdf/bdr11.urdf.xacro (robot description, xacro)
@@ -2,32 +2,12 @@
 <robot xmlns:xacro="http://ros.org/wiki/xacro" name="dual_robots">
   <!-- Define the world link -->
-  <link name="dual_robot_link">
-    <inertial>
-      <mass value="1.0" />
-      <origin xyz="0 0 0.0" rpy="0 0 0" /> <!-- Raise the link by changing the z-value -->
-      <inertia ixx="0" ixy="0" ixz="0" iyy="0" iyz="0" izz="0" />
-    </inertial>
-    <visual>
-      <geometry>
-        <box size="0.01 0.01 0.01" />
-      </geometry>
-      <collision>
-          <origin rpy="0 0 0" xyz="0 0 0" />
-          <geometry>
-              <box size="0.01 0.01 0.01" />
-          </geometry>
-      </collision>
-      <material name="gray">
-        <color rgba="0.5 0.5 0.5 1.0" />
-      </material>
-    </visual>
-  </link>
+    <link name="world" />
   <!-- First robot -->
   <xacro:include filename="$(find bdr11_description)/urdf/ur10_robot.xacro" />
   <xacro:ur10_robot />
   <joint name="ur10_robot_joint" type="fixed">
-    <parent link="dual_robot_link" />
+    <parent link="world" />
     <child link="${ur10_ns}table_link" /> <!-- ${ur10_ns} -->
-    <origin xyz="0 0 -0.005" rpy="0 0 0" />
+    <origin xyz="0 0 0" rpy="0 0 0" />
   </joint>
   <!-- Second robot -->
@@ -35,7 +15,7 @@
   <xacro:moveit_quantec />
   <joint name="quantec_robot_joint" type="fixed">
-    <parent link="dual_robot_link" />
+    <parent link="world" />
     <child link="${quantec_ns}base_link_quantec" />  <!-- ${quantec_ns} -->
-    <origin xyz="-1 0.4 -0.005" rpy="-1.57 0 0" /> <!-- Adjust xyz for the desired position -->
+    <origin xyz="-1 0.4 0" rpy="-1.57 0 0" /> <!-- Adjust xyz for the desired position -->
   </joint>
 </robot>

File: src/bdr11_moveit_config_v1/config/gazebo_dual_robots.urdf (robot description, URDF)
Before this commit: robot dual_robots, 26 links, 25 joints
Links:
- removed link dual_robot_link
- added link world
- link camera_link: geometry collision mesh filename=package://ur10_description_v3/meshes/camera_link.STL; visual mesh filename=package://ur10_description_v3/meshes/camera_link.STL
Joints:
- joint quantec_robot_joint: origin xyz=-1 0.4 -0.005 rpy=-1.57 0 0 -> xyz=-1 0.4 0 rpy=-1.57 0 0; parent dual_robot_link -> world
- joint ur10_robot_joint: origin xyz=0 0 -0.005 rpy=0 0 0 -> xyz=0 0 0 rpy=0 0 0; parent dual_robot_link -> world
